Commit message: Simplifications by maros and renaming

File: robotiq_description/urdf/robotiq_85.urdf.xacro (robot description, xacro)
@@ -1,5 +1,5 @@
 <?xml version="1.0" ?>
-<robot name="robotiq_85_gripper" xmlns:xacro="http://www.ros.org/wiki/xacro">
-  <xacro:include filename="$(find robotiq_description)/urdf/robotiq_85_gripper.urdf.xacro" />
+<robot name="robotiq_85" xmlns:xacro="http://www.ros.org/wiki/xacro">
+  <xacro:include filename="$(find robotiq_description)/urdf/robotiq_85.xacro" />
   <gazebo>
     <plugin name="gazebo_ros_control" filename="libgazebo_ros_control.so">
@@ -11,7 +11,7 @@
     <origin xyz="0 0 0" rpy="0 0 0"/>
     <parent link="world"/>
-    <child link="gripper_root_link"/>
+    <child link="robotiq_85_root_link"/>
   </joint>
-  <link name="gripper_root_link">
+  <link name="robotiq_85_root_link">
     <visual>
       <origin xyz="0 0 0.5" rpy="0 0 0"/>
@@ -34,6 +34,6 @@
     </inertial>
   </link>
-  <xacro:robotiq_85_gripper prefix="" parent="gripper_root_link" >
-    <origin xyz="0.05 0 0.85" rpy="0 0 0"/>
-  </xacro:robotiq_85_gripper>
+  <xacro:robotiq_85 prefix="" parent="robotiq_85_root_link" >
+    <origin xyz="0.05 0 0.robotiq_85" rpy="0 0 0"/>
+  </xacro:robotiq_85>
 </robot>

File: robotiq_description/urdf/robotiq_85.xacro (robot description, xacro)
@@ -1,6 +1,5 @@
 <?xml version="1.0"?>
-<robot name="robotiq_85_gripper" xmlns:xacro="http://www.ros.org/wiki/xacro">
-  <xacro:include filename="$(find robotiq_description)/urdf/robotiq_85_gripper.transmission.xacro" />
-  <xacro:macro name="robotiq_85_gripper" params="prefix parent *origin">
+<robot xmlns:xacro="http://www.ros.org/wiki/xacro" name="robotiq_85">
+  <xacro:macro name="robotiq_85" params="prefix parent *origin">
     <joint name="${prefix}robotiq_85_base_joint" type="fixed">
       <parent link="${parent}"/>
@@ -11,10 +10,10 @@
       <visual>
         <geometry>
-          <mesh filename="package://robotiq_description/meshes/visual/robotiq_85_base_link.dae"/>
-        </geometry>
-      </visual>
-      <collision>
-        <geometry>
-          <mesh filename="package://robotiq_description/meshes/collision/robotiq_85_base_link.stl"/>
+          <mesh filename="package://robotiq_description/meshes/robotiq_85/visual/base.dae"/>
+        </geometry>
+      </visual>
+      <collision>
+        <geometry>
+          <mesh filename="package://robotiq_description/meshes/robotiq_85/collision/base.stl"/>
         </geometry>
       </collision>
@@ -45,10 +44,10 @@
       <visual>
         <geometry>
-          <mesh filename="package://robotiq_description/meshes/visual/robotiq_85_knuckle_link.dae"/>
-        </geometry>
-      </visual>
-      <collision>
-        <geometry>
-          <mesh filename="package://robotiq_description/meshes/collision/robotiq_85_knuckle_link.stl"/>
+          <mesh filename="package://robotiq_description/meshes/robotiq_85/visual/knuckle.dae"/>
+        </geometry>
+      </visual>
+      <collision>
+        <geometry>
+          <mesh filename="package://robotiq_description/meshes/robotiq_85/collision/knuckle.stl"/>
         </geometry>
       </collision>
@@ -64,10 +63,10 @@
       <visual>
         <geometry>
-          <mesh filename="package://robotiq_description/meshes/visual/robotiq_85_knuckle_link.dae"/>
-        </geometry>
-      </visual>
-      <collision>
-        <geometry>
-          <mesh filename="package://robotiq_description/meshes/collision/robotiq_85_knuckle_link.stl"/>
+          <mesh filename="package://robotiq_description/meshes/robotiq_85/visual/knuckle.dae"/>
+        </geometry>
+      </visual>
+      <collision>
+        <geometry>
+          <mesh filename="package://robotiq_description/meshes/robotiq_85/collision/knuckle.stl"/>
         </geometry>
       </collision>
@@ -93,10 +92,10 @@
       <visual>
         <geometry>
-          <mesh filename="package://robotiq_description/meshes/visual/robotiq_85_finger_link.dae"/>
-        </geometry>
-      </visual>
-      <collision>
-        <geometry>
-          <mesh filename="package://robotiq_description/meshes/collision/robotiq_85_finger_link.stl"/>
+          <mesh filename="package://robotiq_description/meshes/robotiq_85/visual/finger.dae"/>
+        </geometry>
+      </visual>
+      <collision>
+        <geometry>
+          <mesh filename="package://robotiq_description/meshes/robotiq_85/collision/finger.stl"/>
         </geometry>
       </collision>
@@ -112,10 +111,10 @@
       <visual>
         <geometry>
-          <mesh filename="package://robotiq_description/meshes/visual/robotiq_85_finger_link.dae"/>
-        </geometry>
-      </visual>
-      <collision>
-        <geometry>
-          <mesh filename="package://robotiq_description/meshes/collision/robotiq_85_finger_link.stl"/>
+          <mesh filename="package://robotiq_description/meshes/robotiq_85/visual/finger.dae"/>
+        </geometry>
+      </visual>
+      <collision>
+        <geometry>
+          <mesh filename="package://robotiq_description/meshes/robotiq_85/collision/finger.stl"/>
         </geometry>
       </collision>
@@ -128,7 +127,7 @@
       </inertial>
     </link>
-    <joint name="${prefix}robotiq_85_left_inner_knuckle_joint" type="continuous">
-      <parent link="${prefix}robotiq_85_base_link"/>
-      <child link="${prefix}robotiq_85_left_inner_knuckle_link"/>
+    <joint name="${prefix}robotiq_85_left_knuckle_inner_joint" type="continuous">
+      <parent link="${prefix}robotiq_85_base_link"/>
+      <child link="${prefix}robotiq_85_left_knuckle_inner_link"/>
       <axis xyz="0 0 1"/>
       <origin xyz="0.06142 0.0127 0" rpy="${pi} 0.0 0.0" />
@@ -136,7 +135,7 @@
       <mimic joint="${prefix}robotiq_85_left_knuckle_joint" offset="0"/>
     </joint>
-    <joint name="${prefix}robotiq_85_right_inner_knuckle_joint" type="continuous">
-      <parent link="${prefix}robotiq_85_base_link"/>
-      <child link="${prefix}robotiq_85_right_inner_knuckle_link"/>
+    <joint name="${prefix}robotiq_85_right_knuckle_inner_joint" type="continuous">
+      <parent link="${prefix}robotiq_85_base_link"/>
+      <child link="${prefix}robotiq_85_right_knuckle_inner_link"/>
       <axis xyz="0 0 1"/>
       <origin xyz="0.06142 -0.0127 0" rpy="0 0 0"/>
@@ -144,13 +143,13 @@
       <mimic joint="${prefix}robotiq_85_left_knuckle_joint" offset="0"/>
     </joint>
-    <link name="${prefix}robotiq_85_left_inner_knuckle_link">
-      <visual>
-        <geometry>
-          <mesh filename="package://robotiq_description/meshes/visual/robotiq_85_inner_knuckle_link.dae"/>
-        </geometry>
-      </visual>
-      <collision>
-        <geometry>
-          <mesh filename="package://robotiq_description/meshes/collision/robotiq_85_inner_knuckle_link.stl"/>
+    <link name="${prefix}robotiq_85_left_knuckle_inner_link">
+      <visual>
+        <geometry>
+          <mesh filename="package://robotiq_description/meshes/robotiq_85/visual/knuckle_inner.dae"/>
+        </geometry>
+      </visual>
+      <collision>
+        <geometry>
+          <mesh filename="package://robotiq_description/meshes/robotiq_85/collision/knuckle_inner.stl"/>
         </geometry>
       </collision>
@@ -163,13 +162,13 @@
       </inertial>
     </link>
-    <link name="${prefix}robotiq_85_right_inner_knuckle_link">
-      <visual>
-        <geometry>
-          <mesh filename="package://robotiq_description/meshes/visual/robotiq_85_inner_knuckle_link.dae"/>
-        </geometry>
-      </visual>
-      <collision>
-        <geometry>
-          <mesh filename="package://robotiq_description/meshes/collision/robotiq_85_inner_knuckle_link.stl"/>
+    <link name="${prefix}robotiq_85_right_knuckle_inner_link">
+      <visual>
+        <geometry>
+          <mesh filename="package://robotiq_description/meshes/robotiq_85/visual/knuckle_inner.dae"/>
+        </geometry>
+      </visual>
+      <collision>
+        <geometry>
+          <mesh filename="package://robotiq_description/meshes/robotiq_85/collision/knuckle_inner.stl"/>
         </geometry>
       </collision>
@@ -182,7 +181,7 @@
       </inertial>
     </link>
-    <joint name="${prefix}robotiq_85_left_finger_tip_joint" type="continuous">
-      <parent link="${prefix}robotiq_85_left_inner_knuckle_link"/>
-      <child link="${prefix}robotiq_85_left_finger_tip_link"/>
+    <joint name="${prefix}robotiq_85_left_tip_joint" type="continuous">
+      <parent link="${prefix}robotiq_85_left_knuckle_inner_link"/>
+      <child link="${prefix}robotiq_85_left_tip_link"/>
       <axis xyz="0 0 1"/>
       <origin xyz="0.04303959807 -0.03759940821 0.0" rpy="0.0 0.0 0.0"/>
@@ -190,7 +189,7 @@
       <mimic joint="${prefix}robotiq_85_left_knuckle_joint" multiplier="-1"/>
     </joint>
-    <joint name="${prefix}robotiq_85_right_finger_tip_joint" type="continuous">
-      <parent link="${prefix}robotiq_85_right_inner_knuckle_link"/>
-      <child link="${prefix}robotiq_85_right_finger_tip_link"/>
+    <joint name="${prefix}robotiq_85_right_tip_joint" type="continuous">
+      <parent link="${prefix}robotiq_85_right_knuckle_inner_link"/>
+      <child link="${prefix}robotiq_85_right_tip_link"/>
       <axis xyz="0 0 1"/>
       <origin rpy="0.0 0.0 0.0" xyz="0.04303959807 -0.03759940821  0.0"/>
@@ -198,13 +197,13 @@
       <mimic joint="${prefix}robotiq_85_left_knuckle_joint" multiplier="-1"/>
     </joint>
-    <link name="${prefix}robotiq_85_left_finger_tip_link">
-      <visual>
-        <geometry>
-          <mesh filename="package://robotiq_description/meshes/visual/robotiq_85_finger_tip_link.dae"/>
-        </geometry>
-      </visual>
-      <collision>
-        <geometry>
-          <mesh filename="package://robotiq_description/meshes/collision/robotiq_85_finger_tip_link.stl"/>
+    <link name="${prefix}robotiq_85_left_tip_link">
+      <visual>
+        <geometry>
+          <mesh filename="package://robotiq_description/meshes/robotiq_85/visual/tip.dae"/>
+        </geometry>
+      </visual>
+      <collision>
+        <geometry>
+          <mesh filename="package://robotiq_description/meshes/robotiq_85/collision/tip.stl"/>
         </geometry>
       </collision>
@@ -217,13 +216,13 @@
       </inertial>
     </link>
-    <link name="${prefix}robotiq_85_right_finger_tip_link">
-      <visual>
-        <geometry>
-          <mesh filename="package://robotiq_description/meshes/visual/robotiq_85_finger_tip_link.dae"/>
-        </geometry>
-      </visual>
-      <collision>
-        <geometry>
-          <mesh filename="package://robotiq_description/meshes/collision/robotiq_85_finger_tip_link.stl"/>
+    <link name="${prefix}robotiq_85_right_tip_link">
+      <visual>
+        <geometry>
+          <mesh filename="package://robotiq_description/meshes/robotiq_85/visual/tip.dae"/>
+        </geometry>
+      </visual>
+      <collision>
+        <geometry>
+          <mesh filename="package://robotiq_description/meshes/robotiq_85/collision/tip.stl"/>
         </geometry>
       </collision>
@@ -237,5 +236,5 @@
     </link>
     <!-- Improve grasping physics -->
-    <gazebo reference="${prefix}robotiq_85_left_finger_tip_link">
+    <gazebo reference="${prefix}robotiq_85_left_tip_link">
       <kp>1000000.0</kp>
       <kd>1.0</kd>
@@ -244,5 +243,5 @@
       <minDepth>0.001</minDepth>
     </gazebo>
-    <gazebo reference="${prefix}robotiq_85_right_finger_tip_link">
+    <gazebo reference="${prefix}robotiq_85_right_tip_link">
       <kp>1000000.0</kp>
       <kd>1.0</kd>
@@ -251,5 +250,41 @@
       <minDepth>0.001</minDepth>
     </gazebo>
-    <xacro:robotiq_85_gripper_transmission prefix="${prefix}" />
+    <transmission name="${prefix}robotiq_85_left_knuckle_trans">
+      <type>transmission_interface/SimpleTransmission</type>
+      <joint name="${prefix}robotiq_85_left_knuckle_joint">
+        <hardwareInterface>hardware_interface/PositionJointInterface</hardwareInterface>
+      </joint>
+      <actuator name="${prefix}robotiq_85_left_knuckle_motor">
+        <mechanicalReduction>1</mechanicalReduction>
+        <hardwareInterface>hardware_interface/PositionJointInterface</hardwareInterface>
+      </actuator>
+    </transmission>
+    <!-- Mimic joints -->
+    <gazebo>
+      <plugin filename="libroboticsgroup_upatras_gazebo_mimic_joint_plugin.so" name="${prefix}mimic_robotiq_85_1">
+        <joint>${prefix}robotiq_85_left_knuckle_joint</joint>
+        <mimicJoint>${prefix}robotiq_85_right_knuckle_joint</mimicJoint>
+      </plugin>
+      <plugin filename="libroboticsgroup_upatras_gazebo_mimic_joint_plugin.so" name="${prefix}mimic_robotiq_85_2">
+        <joint>${prefix}robotiq_85_left_knuckle_joint</joint>
+        <mimicJoint>${prefix}robotiq_85_left_knuckle_inner_joint</mimicJoint>
+      </plugin>
+      <plugin filename="libroboticsgroup_upatras_gazebo_mimic_joint_plugin.so" name="${prefix}mimic_robotiq_85_3">
+        <joint>${prefix}robotiq_85_left_knuckle_joint</joint>
+        <mimicJoint>${prefix}robotiq_85_right_knuckle_inner_joint</mimicJoint>
+      </plugin>
+      <plugin filename="libroboticsgroup_upatras_gazebo_mimic_joint_plugin.so" name="${prefix}mimic_robotiq_85_4">
+        <joint>${prefix}robotiq_85_left_knuckle_joint</joint>
+        <mimicJoint>${prefix}robotiq_85_left_tip_joint</mimicJoint>
+        <multiplier>-1.0</multiplier>
+        <offset>0.0</offset>
+      </plugin>
+      <plugin filename="libroboticsgroup_upatras_gazebo_mimic_joint_plugin.so" name="${prefix}mimic_robotiq_85_5">
+        <joint>${prefix}robotiq_85_left_knuckle_joint</joint>
+        <mimicJoint>${prefix}robotiq_85_right_tip_joint</mimicJoint>
+        <multiplier>-1.0</multiplier>
+        <offset>0.0</offset>
+      </plugin>
+    </gazebo>
   </xacro:macro>
 </robot>

File: robotiq_description/urdf/robotiq_85_sim_base.urdf.xacro (robot description, xacro)
@@ -1,6 +1,6 @@
 <?xml version="1.0"?>
-<robot name="robotiq_85_gripper_sim_base" xmlns:xacro="http://www.ros.org/wiki/xacro">
-  <xacro:macro name="robotiq_85_gripper_sim_base" params="prefix">
-    <link name="${prefix}gripper_root_link">
+<robot name="robotiq_85_sim_base" xmlns:xacro="http://www.ros.org/wiki/xacro">
+  <xacro:macro name="robotiq_85_sim_base" params="prefix">
+    <link name="${prefix}robotiq_85_root_link">
       <visual>
         <origin xyz="0.05 0.05 0.5" rpy="0 0 0"/>
